Commit message: Renamed link: base -> base_link
Signed-off-by: Juancams <jc.manzanares.serrano@gmail.com>

File: go2_description/urdf/go2_description.urdf (robot description, URDF)
Before this commit: robot go2_description, 29 links, 28 joints
Links:
- removed link base
- added link base_link, mass 6.921; collision box size=0.3762 0.0935 0.114; visual mesh filename=package://go2_description/dae/base.dae
Joints:
- joint FL_hip_joint: parent base -> base_link
- joint FR_hip_joint: parent base -> base_link
- joint Head_upper_joint: parent base -> base_link
- joint RL_hip_joint: parent base -> base_link
- joint RR_hip_joint: parent base -> base_link
- joint imu_joint: parent base -> base_link
- joint radar_joint: parent base -> base_link

Commit message: Changed URDF to add hsai laser and realsense camer
Added in the urdf the tf of realsense camera and hsai laser in order to avoid publishing a tf static transform

File: go2_description/urdf/go2_description.urdf (robot description, URDF)
Before this commit: robot go2_description, 29 links, 28 joints
Links:
- removed link base_link
- added link base, mass 6.921; collision box size=0.3762 0.0935 0.114; visual mesh filename=package://go2_description/dae/base.dae
- added link camera_link; collision cylinder length=0.09 radius=0.05; visual cylinder length=0.01 radius=0.01
- added link hesai_lidar; collision cylinder length=0.09 radius=0.05; visual cylinder length=0.09 radius=0.05
Joints:
- added joint camera_link_joint: type fixed, parent {robot_num}/front_camera, child camera_link, origin xyz=0 -0.05 0 rpy=0 0 0, axis 0 0 0
- added joint hesai_lidar_joint: type fixed, parent {robot_num}/base_link, child hesai_lidar, origin xyz=0.15 0 0.08 rpy=1.56 0 0, axis 0 0 0
- joint FL_hip_joint: parent base_link -> base
- joint FR_hip_joint: parent base_link -> base
- joint Head_upper_joint: parent base_link -> base
- joint RL_hip_joint: parent base_link -> base
- joint RR_hip_joint: parent base_link -> base
- joint imu_joint: parent base_link -> base
- joint radar_joint: parent base_link -> base
